File: i2c/diagram/i2c.kicad_sch (KiCad schematic)
At the start: 1 part

Commit message: update i2c
Parts:
- added R1, R2: 3k3, symbol Device:R
Connections:
- net SCL: now also R1.2
- net SDA: now also R2.2
- net +3.3V: now reaches U1.00 (3V3)
- net +3.3V: now also R1.1, R2.1
- net GND: now reaches U1.0C (GND)
Other:
- moved on the sheet: U1
